Commit message: add a camera

File: src/hardware/hardware_core/urdf/components/sensors/livox_mid_360.xacro (robot description, xacro)
@@ -2,5 +2,5 @@
 <robot xmlns:xacro="http://www.ros.org/wiki/xacro">
     <xacro:include filename="$(find hardware_core)/urdf/helpers/materials.xacro" />
-    <xacro:macro name="livox_mid_360" params="name parent xyz rpy">
+    <xacro:macro name="livox_mid_360" params="name parent xyz rpy='0 0 0'">
         <joint name="livox_${name}_joint" type="fixed">
             <parent link="${parent}" />

File: src/hardware/hardware_core/urdf/racecar.urdf.xacro (robot description, xacro)
@@ -5,4 +5,5 @@
     <xacro:include filename="$(find hardware_core)/urdf/components/wheel_rear.xacro" />
     <xacro:include filename="$(find hardware_core)/urdf/components/sensors/livox_mid_360.xacro" />
+    <xacro:include filename="$(find hardware_core)/urdf/components/sensors/camera.xacro" />
     <link name="base_link" />
     <xacro:chassis parent="base_link" xyz="0 0 0" />
@@ -11,3 +12,4 @@
     <xacro:wheel_rear name="right" parent="chassis" xyz="-4.21 -0.772 0" />
     <xacro:livox_mid_360 name="front" parent="chassis" xyz="-2.39 0 0.8" rpy="${pi} 0 0"/>
+    <xacro:camera name="front" parent="chassis" xyz="-2.39 0 0.85"/>
 </robot>

File: src/hardware/hardware_gazebo/urdf/racecar.urdf.xacro (robot description, xacro)
@@ -2,8 +2,10 @@
 <robot xmlns:xacro="http://www.ros.org/wiki/xacro" name="racecar">
     <xacro:include filename="$(find hardware_gazebo)/urdf/components/sensors/livox_mid_360.xacro" />
-    <xacro:include filename="$(find hardware_core)/urdf/racecar.urdf.xacro" />
+    <xacro:include filename="$(find hardware_gazebo)/urdf/components/sensors/camera.xacro" />
     <xacro:include filename="$(find hardware_gazebo)/urdf/components/gz_ros2_control.urdf.xacro" />
     <xacro:include filename="$(find hardware_gazebo)/urdf/components/ros2_control.urdf.xacro" />
     <xacro:include filename="$(find hardware_gazebo)/urdf/components/sensor_plugin.urdf.xacro" />
+    <xacro:include filename="$(find hardware_core)/urdf/racecar.urdf.xacro" />
     <xacro:gz_livox_mid_360 name="front" />
+    <xacro:gz_camera name="front" />
 </robot>
